Commit message: fix(urdf): 修正夹爪关节轴方向和限位，添加默认关节状态
调整了左右夹爪的关节旋转轴方向与关节限位范围，同时为两个夹爪的关节添加了手指完全张开的默认初始状态

File: assets/zerith/urdf/left_gripper.urdf (robot description, URDF)
Before this commit: robot zerith_left_gripper, 6 links, 5 joints
Joints:
- joint left_jaw_right_finger_joint: axis 0 1 0 -> 0 -1 0; limit lower=0 upper=0.04 effort=120 velocity=0.25 -> lower=-0.04 upper=0 effort=120 velocity=0.25

File: assets/zerith/urdf/right_gripper.urdf (robot description, URDF)
Before this commit: robot zerith_right_gripper, 6 links, 5 joints
Joints:
- joint right_jaw_left_finger_joint: axis 0 1 0 -> 0 -1 0
