Commit message: fix(urdf): 修正右夹爪关节的轴方向和运动限位范围
调整right_gripper.urdf中右夹爪关节的axis参数为0 -1 0，同时将关节限位的上下限从0到0.04改为-0.04到0，匹配实际开合运动逻辑

File: assets/zerith/urdf/right_gripper.urdf (robot description, URDF)
Before this commit: robot zerith_right_gripper, 6 links, 5 joints
Joints:
- joint right_jaw_right_finger_joint: axis 0 1 0 -> 0 -1 0; limit lower=0 upper=0.04 effort=120 velocity=0.25 -> lower=-0.04 upper=0 effort=120 velocity=0.25

Commit message: fix(urdf,tools): 修正右夹爪关节轴方向并固定夹具配置向导名称
1.  修正right_gripper.urdf的关节轴xyz参数为0 1 0，修复夹爪开合方向错误
2.  固定run_gripper_config_wizard.sh中的左右夹爪名称为固定值，替代原动态取文件名逻辑

File: assets/zerith/urdf/right_gripper.urdf (robot description, URDF)
Before this commit: robot zerith_right_gripper, 6 links, 5 joints
Joints:
- joint right_jaw_left_finger_joint: axis 0 -1 0 -> 0 1 0
